Commit message: replace main urdf with new model and remove old assets

File: src/sukinee_urdf/urdf/sukinee_urdf.urdf (robot description, URDF)
Before this commit: robot sukinee_urdf, 11 links, 10 joints
Links:
- added link world
- link Link1: mass 0.173424729959474 -> 0.173656729959474; geometry collision mesh filename=package://sukinee_urdf/meshes/urdf2/Link1.STL; visual mesh filename=package://sukinee_urdf/meshes/urdf2/Link1.STL
- link Link10: mass 0.0514991248787955 -> 0.0483309609625738; geometry collision mesh filename=package://sukinee_urdf/meshes/urdf2/left_Link.STL; visual mesh filename=package://sukinee_urdf/meshes/urdf2/left_Link.STL
- link Link2: mass 0.49221073789159 -> 0.486273817491279; geometry collision mesh filename=package://sukinee_urdf/meshes/urdf2/Link2.STL; visual mesh filename=package://sukinee_urdf/meshes/urdf2/Link2.STL
- link Link3: mass 0.342921181307181 -> 0.324306511251341; geometry collision mesh filename=package://sukinee_urdf/meshes/urdf2/Link3.STL; visual mesh filename=package://sukinee_urdf/meshes/urdf2/Link3.STL
- link Link4: mass 0.0535059280721223 -> 0.058588375547201; geometry collision mesh filename=package://sukinee_urdf/meshes/urdf2/Link4.STL; visual mesh filename=package://sukinee_urdf/meshes/urdf2/Link4.STL
- link Link5: mass 0.042177959365491 -> 0.0484344180023895; geometry collision mesh filename=package://sukinee_urdf/meshes/urdf2/Link5.STL; visual mesh filename=package://sukinee_urdf/meshes/urdf2/Link5.STL
- link Link6: mass 0.10618748414872 -> 0.159442082245761; geometry collision mesh filename=package://sukinee_urdf/meshes/urdf2/Link6.STL; visual mesh filename=package://sukinee_urdf/meshes/urdf2/Link6.STL
- link Link7: mass 0.0056954950921208 -> 0.00564266139065291; geometry collision mesh filename=package://sukinee_urdf/meshes/urdf2/Link7.STL; visual mesh filename=package://sukinee_urdf/meshes/urdf2/Link7.STL
- link Link8: mass 0.0685515728356248 -> 0.0196144070602556; geometry collision mesh filename=package://sukinee_urdf/meshes/urdf2/Link8.STL; visual mesh filename=package://sukinee_urdf/meshes/urdf2/Link8.STL
- link Link9: mass 0.0514991247749255 -> 0.0483309612331933; geometry collision mesh filename=package://sukinee_urdf/meshes/urdf2/right_Link.STL; visual mesh filename=package://sukinee_urdf/meshes/urdf2/right_Link.STL
- link base_link: mass 0.276557659513136 -> 0.258345451540463; geometry collision mesh filename=package://sukinee_urdf/meshes/urdf2/base_link.STL; visual mesh filename=package://sukinee_urdf/meshes/urdf2/base_link.STL
Joints:
- added joint world_to_base_link: type fixed, parent world, child base_link, origin xyz=0 0 0.0 rpy=0 0 0
- joint Joint1: axis 0 0 1 -> 0 0 -1; origin xyz=-4.5606E-05 -0.00029999 0.051399 rpy=0 0 0 -> xyz=0 0 0.0514 rpy=0 0 0
- joint Joint2: axis 0 0 1 -> 0 0 -1; origin xyz=0.0068769 -0.027546 0.042346 rpy=-1.5708 0 3.1416 -> xyz=-0.010939 0.025949 0.0425 rpy=-1.5708 -0.00097565 0.16603
- joint Joint3: axis 0 0 1 -> 0 0 -1; origin xyz=0.26443 0.0031418 0.0039907 rpy=0 0 0 -> xyz=0.26636 0.0076666 0 rpy=0 0 0
- joint Joint4: axis 0 0 1 -> 0 0 -1; origin xyz=-0.24836 -0.068439 -0.0072675 rpy=0 0 3.1416 -> xyz=-0.25125 -0.065507 -0.0039 rpy=0 0 0
- joint Joint5: axis 0 0 1 -> 0 0 -1; origin xyz=0.061641 0.045136 -0.024175 rpy=1.5708 0 0 -> xyz=-0.059809 -0.047874 -0.0245 rpy=1.5708 -1.448 -3.0944
- joint Joint6: axis 0 0 1 -> 0 0 -1; limit lower=-0.79 upper=0.79 effort=1.6 velocity=3.14 -> effort=1.6 velocity=3.14; origin xyz=0.019993 -0.00056516 0.044999 rpy=1.5708 0 1.5708 -> xyz=0.00093628 -0.019978 0.045 rpy=1.5708 0.0022273 0.046831
- joint Joint7: axis 0 0 1 -> 0 0 -1; origin xyz=0.00010901 0.00023352 -0.016998 rpy=0 0 1.1345 -> xyz=0.0015425 0.00080701 -0.016911 rpy=0.047489 -0.090961 0
- joint Joint8: origin xyz=-0.0011196 0.00014947 0.074992 rpy=0 0 -1.1345 -> xyz=1.7949E-05 0.00014892 0.075 rpy=-0.047686 0.090858 -0.00433
- joint left_finger: limit lower=-0.006 upper=0.006 effort=1 velocity=0.05 -> lower=0 upper=0.04 effort=1 velocity=0.03; mimic joint=Joint7 multiplier=0.02 offset=0 -> joint=Joint7 multiplier=0.05 offset=0; origin xyz=0.00079796 0.041726 0.0087023 rpy=-2.7256 -1.5556 -2.0071 -> xyz=-0.038848 -0.01714 0.0038046 rpy=-0.41189 1.4591 0
- joint right_finger: limit lower=-0.006 upper=0.006 effort=1 velocity=0.05 -> lower=0 upper=0.04 effort=1 velocity=0.03; mimic joint=Joint7 multiplier=0.02 offset=0 -> joint=Joint7 multiplier=0.05 offset=0; origin xyz=-0.00090214 -0.041949 0.0075419 rpy=-0.41597 1.5556 1.1345 -> xyz=0.037374 0.016369 0.012356 rpy=-2.7297 -1.4591 3.1416

File: src/sukinee_urdf/urdf/sukinee_urdf.urdf.xacro (robot description, xacro)
@@ -19,37 +19,37 @@
     <inertial>
       <origin
-        xyz="-9.27159793573523E-05 5.84334903300024E-05 0.0131634742942032"
-        rpy="0 0 0" />
-      <mass
-        value="0.276557659513136" />
-      <inertia
-        ixx="0.000306944214419235"
-        ixy="-2.62966486226292E-05"
-        ixz="-2.17057678389435E-07"
-        iyy="0.00019619720224458"
-        iyz="-1.11233404518986E-06"
-        izz="0.000381711312546233" />
-    </inertial>
-    <visual>
-      <origin
-        xyz="0 0 0"
-        rpy="0 0 0" />
-      <geometry>
-        <mesh
-          filename="package://sukinee_urdf/meshes/base_link.STL" />
-      </geometry>
-      <material
-        name="">
-        <color
-          rgba="1 1 1 1" />
-      </material>
-    </visual>
-    <collision>
-      <origin
-        xyz="0 0 0"
-        rpy="0 0 0" />
-      <geometry>
-        <mesh
-          filename="package://sukinee_urdf/meshes/base_link.STL" />
+        xyz="1.32130893254478E-07 1.0878882315303E-07 0.0145123930882944"
+        rpy="0 0 0" />
+      <mass
+        value="0.258345451540463" />
+      <inertia
+        ixx="0.000255695833262824"
+        ixy="-8.50566806153412E-06"
+        ixz="6.25989218367775E-10"
+        iyy="0.000143791450764687"
+        iyz="5.1542362971656E-10"
+        izz="0.0003184122634403" />
+    </inertial>
+    <visual>
+      <origin
+        xyz="0 0 0"
+        rpy="0 0 0" />
+      <geometry>
+        <mesh
+          filename="package://sukinee_urdf/meshes/urdf2/base_link.STL" />
+      </geometry>
+      <material
+        name="">
+        <color
+          rgba="1 1 1 1" />
+      </material>
+    </visual>
+    <collision>
+      <origin
+        xyz="0 0 0"
+        rpy="0 0 0" />
+      <geometry>
+        <mesh
+          filename="package://sukinee_urdf/meshes/urdf2/base_link.STL" />
       </geometry>
     </collision>
@@ -59,37 +59,37 @@
     <inertial>
       <origin
-        xyz="0.00328193566941784 -0.00101264174932876 0.0341645293592959"
-        rpy="0 0 0" />
-      <mass
-        value="0.173424729959474" />
-      <inertia
-        ixx="8.50037683173789E-05"
-        ixy="2.28577329805091E-07"
-        ixz="-7.19620303243764E-07"
-        iyy="7.01795557782873E-05"
-        iyz="-1.21785758387906E-07"
-        izz="8.92996495432085E-05" />
-    </inertial>
-    <visual>
-      <origin
-        xyz="0 0 0"
-        rpy="0 0 0" />
-      <geometry>
-        <mesh
-          filename="package://sukinee_urdf/meshes/Link1.STL" />
-      </geometry>
-      <material
-        name="">
-        <color
-          rgba="1 1 1 1" />
-      </material>
-    </visual>
-    <collision>
-      <origin
-        xyz="0 0 0"
-        rpy="0 0 0" />
-      <geometry>
-        <mesh
-          filename="package://sukinee_urdf/meshes/Link1.STL" />
+        xyz="-0.00339213548156639 0.000304711073311301 0.034122625208467"
+        rpy="0 0 0" />
+      <mass
+        value="0.173656729959474" />
+      <inertia
+        ixx="8.56959788246817E-05"
+        ixy="2.57981779041257E-06"
+        ixz="7.14608803543954E-07"
+        iyy="7.07301657377921E-05"
+        iyz="1.19276284474143E-07"
+        izz="9.04237787575582E-05" />
+    </inertial>
+    <visual>
+      <origin
+        xyz="0 0 0"
+        rpy="0 0 0" />
+      <geometry>
+        <mesh
+          filename="package://sukinee_urdf/meshes/urdf2/Link1.STL" />
+      </geometry>
+      <material
+        name="">
+        <color
+          rgba="1 1 1 1" />
+      </material>
+    </visual>
+    <collision>
+      <origin
+        xyz="0 0 0"
+        rpy="0 0 0" />
+      <geometry>
+        <mesh
+          filename="package://sukinee_urdf/meshes/urdf2/Link1.STL" />
       </geometry>
     </collision>
@@ -97,7 +97,7 @@
   <joint
     name="Joint1"
-    type="revolute">
-    <origin
-      xyz="-4.5606E-05 -0.00029999 0.051399"
+    type="continuous">
+    <origin
+      xyz="0 0 0.0514"
       rpy="0 0 0" />
     <parent
@@ -106,8 +106,6 @@
       link="Link1" />
     <axis
-      xyz="0 0 1" />
-    <limit
-      lower="-3.1416"
-      upper="3.1416"
+      xyz="0 0 -1" />
+    <limit
       effort="5"
       velocity="3.14" />
@@ -117,37 +115,37 @@
     <inertial>
       <origin
-        xyz="0.163147205394747 0.0077249837082756 -0.0251647837081496"
-        rpy="0 0 0" />
-      <mass
-        value="0.49221073789159" />
-      <inertia
-        ixx="0.00013320567604932"
-        ixy="-1.90333861615628E-05"
-        ixz="-2.02132460329359E-05"
-        iyy="0.00146041125210994"
-        iyz="-3.49082300685114E-07"
-        izz="0.00147443591285137" />
-    </inertial>
-    <visual>
-      <origin
-        xyz="0 0 0"
-        rpy="0 0 0" />
-      <geometry>
-        <mesh
-          filename="package://sukinee_urdf/meshes/Link2.STL" />
-      </geometry>
-      <material
-        name="">
-        <color
-          rgba="1 1 1 1" />
-      </material>
-    </visual>
-    <collision>
-      <origin
-        xyz="0 0 0"
-        rpy="0 0 0" />
-      <geometry>
-        <mesh
-          filename="package://sukinee_urdf/meshes/Link2.STL" />
+        xyz="0.164355934511196 0.0107983189121957 -0.0273278206693135"
+        rpy="0 0 0" />
+      <mass
+        value="0.486273817491279" />
+      <inertia
+        ixx="0.000131700208765616"
+        ixy="-3.59955416546668E-05"
+        ixz="-4.49796251556987E-06"
+        iyy="0.00142428639296128"
+        iyz="-7.11032579861893E-07"
+        izz="0.00143980686835948" />
+    </inertial>
+    <visual>
+      <origin
+        xyz="0 0 0"
+        rpy="0 0 0" />
+      <geometry>
+        <mesh
+          filename="package://sukinee_urdf/meshes/urdf2/Link2.STL" />
+      </geometry>
+      <material
+        name="">
+        <color
+          rgba="1 1 1 1" />
+      </material>
+    </visual>
+    <collision>
+      <origin
+        xyz="0 0 0"
+        rpy="0 0 0" />
+      <geometry>
+        <mesh
+          filename="package://sukinee_urdf/meshes/urdf2/Link2.STL" />
       </geometry>
     </collision>
@@ -157,6 +155,6 @@
     type="revolute">
     <origin
-      xyz="0.0068769 -0.027546 0.042346"
-      rpy="-1.5708 0 3.1416" />
+      xyz="-0.010939 0.025949 0.0425"
+      rpy="-1.5708 -0.00097565 0.16603" />
     <parent
       link="Link1" />
@@ -164,5 +162,5 @@
       link="Link2" />
     <axis
-      xyz="0 0 1" />
+      xyz="0 0 -1" />
     <limit
       lower="-0.79"
@@ -175,37 +173,37 @@
     <inertial>
       <origin
-        xyz="-0.123533258510765 -0.0531477412867997 -0.0289818543594236"
-        rpy="0 0 0" />
-      <mass
-        value="0.342921181307181" />
-      <inertia
-        ixx="8.97920455274715E-05"
-        ixy="-5.81304856828259E-05"
-        ixz="-1.06742108487144E-05"
-        iyy="0.00076637159477087"
-        iyz="-9.66346038777982E-07"
-        izz="0.00078459383677109" />
-    </inertial>
-    <visual>
-      <origin
-        xyz="0 0 0"
-        rpy="0 0 0" />
-      <geometry>
-        <mesh
-          filename="package://sukinee_urdf/meshes/Link3.STL" />
-      </geometry>
-      <material
-        name="">
-        <color
-          rgba="1 1 1 1" />
-      </material>
-    </visual>
-    <collision>
-      <origin
-        xyz="0 0 0"
-        rpy="0 0 0" />
-      <geometry>
-        <mesh
-          filename="package://sukinee_urdf/meshes/Link3.STL" />
+        xyz="-0.129522607900688 -0.0521849921825459 -0.0273613995018329"
+        rpy="0 0 0" />
+      <mass
+        value="0.324306511251341" />
+      <inertia
+        ixx="8.179700405764E-05"
+        ixy="-4.69997732333903E-05"
+        ixz="1.35034163751212E-06"
+        iyy="0.000731273265167081"
+        iyz="-3.54063317410718E-07"
+        izz="0.00075003040907452" />
+    </inertial>
+    <visual>
+      <origin
+        xyz="0 0 0"
+        rpy="0 0 0" />
+      <geometry>
+        <mesh
+          filename="package://sukinee_urdf/meshes/urdf2/Link3.STL" />
+      </geometry>
+      <material
+        name="">
+        <color
+          rgba="1 1 1 1" />
+      </material>
+    </visual>
+    <collision>
+      <origin
+        xyz="0 0 0"
+        rpy="0 0 0" />
+      <geometry>
+        <mesh
+          filename="package://sukinee_urdf/meshes/urdf2/Link3.STL" />
       </geometry>
     </collision>
@@ -215,5 +213,5 @@
     type="revolute">
     <origin
-      xyz="0.26443 0.0031418 0.0039907"
+      xyz="0.26636 0.0076666 0"
       rpy="0 0 0" />
     <parent
@@ -222,5 +220,5 @@
       link="Link3" />
     <axis
-      xyz="0 0 1" />
+      xyz="0 0 -1" />
     <limit
       lower="-0.79"
@@ -233,37 +231,37 @@
     <inertial>
       <origin
-        xyz="0.0325057327109481 0.0348518868836431 -0.0264977574735537"
-        rpy="0 0 0" />
-      <mass
-        value="0.0535059280721223" />
-      <inertia
-        ixx="3.35516541099526E-05"
-        ixy="-9.36823847263875E-06"
-        ixz="-1.44258751379024E-07"
-        iyy="4.45006403501621E-05"
-        iyz="9.87407338332834E-08"
-        izz="3.33930480114162E-05" />
-    </inertial>
-    <visual>
-      <origin
-        xyz="0 0 0"
-        rpy="0 0 0" />
-      <geometry>
-        <mesh
-          filename="package://sukinee_urdf/meshes/Link4.STL" />
-      </geometry>
-      <material
-        name="">
-        <color
-          rgba="1 1 1 1" />
-      </material>
-    </visual>
-    <collision>
-      <origin
-        xyz="0 0 0"
-        rpy="0 0 0" />
-      <geometry>
-        <mesh
-          filename="package://sukinee_urdf/meshes/Link4.STL" />
+        xyz="-0.0338567228905684 -0.0377615700439491 -0.0271938522907798"
+        rpy="0 0 0" />
+      <mass
+        value="0.058588375547201" />
+      <inertia
+        ixx="3.47939295698438E-05"
+        ixy="-9.83781789279702E-06"
+        ixz="8.18793872056976E-08"
+        iyy="4.43014363876168E-05"
+        iyz="1.11539635337878E-07"
+        izz="3.36963199084079E-05" />
+    </inertial>
+    <visual>
+      <origin
+        xyz="0 0 0"
+        rpy="0 0 0" />
+      <geometry>
+        <mesh
+          filename="package://sukinee_urdf/meshes/urdf2/Link4.STL" />
+      </geometry>
+      <material
+        name="">
+        <color
+          rgba="1 1 1 1" />
+      </material>
+    </visual>
+    <collision>
+      <origin
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