Commit message: add stable gazebo effort impedance baseline

File: src/sukinee_urdf/urdf/sukinee_ros2_control.xacro (robot description, xacro)
@@ -1,44 +1,44 @@
 <?xml version="1.0"?>
 <robot xmlns:xacro="http://www.ros.org/wiki/xacro">
-  <xacro:macro name="sukinee_ros2_control" params="use_mock_hardware">
+  <xacro:macro name="sukinee_ros2_control" params="use_mock_hardware hardware_plugin arm_command_interface gripper_command_interface">
     <ros2_control name="SukineeSystem" type="system">
-      <hardware>
-        <xacro:if value="${use_mock_hardware}">
-          <plugin>mock_components/GenericSystem</plugin>
-          <param name="mock_sensor_commands">false</param>
-        </xacro:if>
-      </hardware>
+    <hardware>
+      <plugin>${hardware_plugin}</plugin>
+      <xacro:if value="${use_mock_hardware}">
+        <param name="mock_sensor_commands">false</param>
+      </xacro:if>
+    </hardware>
       <joint name="Joint1">
-        <command_interface name="position"/>
+        <command_interface name="${arm_command_interface}"/>
         <state_interface name="position"/>
         <state_interface name="velocity"/>
       </joint>
       <joint name="Joint2">
-        <command_interface name="position"/>
+        <command_interface name="${arm_command_interface}"/>
         <state_interface name="position"/>
         <state_interface name="velocity"/>
       </joint>
       <joint name="Joint3">
-        <command_interface name="position"/>
+        <command_interface name="${arm_command_interface}"/>
         <state_interface name="position"/>
         <state_interface name="velocity"/>
       </joint>
       <joint name="Joint4">
-        <command_interface name="position"/>
+        <command_interface name="${arm_command_interface}"/>
         <state_interface name="position"/>
         <state_interface name="velocity"/>
       </joint>
       <joint name="Joint5">
-        <command_interface name="position"/>
+        <command_interface name="${arm_command_interface}"/>
         <state_interface name="position"/>
         <state_interface name="velocity"/>
       </joint>
       <joint name="Joint6">
-        <command_interface name="position"/>
+        <command_interface name="${arm_command_interface}"/>
         <state_interface name="position"/>
         <state_interface name="velocity"/>
       </joint>
       <joint name="Joint7">
-        <command_interface name="position"/>
+        <command_interface name="${gripper_command_interface}"/>
         <state_interface name="position"/>
         <state_interface name="velocity"/>

File: src/sukinee_urdf/urdf/sukinee_urdf.urdf.xacro (robot description, xacro)
@@ -2,4 +2,10 @@
 <robot name="sukinee_urdf" xmlns:xacro="http://www.ros.org/wiki/xacro">
   <xacro:arg name="use_mock_hardware" default="true"/>
+  <xacro:arg name="hardware_plugin" default="mock_components/GenericSystem"/>
+  <xacro:arg name="arm_command_interface" default="position"/>
+  <xacro:arg name="gripper_command_interface" default="position"/>
+  <xacro:arg name="include_gz_plugin" default="false"/>
+  <xacro:arg name="controllers_file" default=""/>
+  <xacro:arg name="world_z" default="0.0"/>
   <xacro:include filename="$(find sukinee_urdf)/urdf/sukinee_ros2_control.xacro"/>
   <link name="world"/>
@@ -7,5 +13,5 @@
     <parent link="world"/>
     <child link="base_link"/>
-    <origin xyz="0 0 0" rpy="0 0 0"/>
+    <origin xyz="0 0 $(arg world_z)" rpy="0 0 0"/>
   </joint>
   <link
@@ -632,4 +638,15 @@
       offset="0" />
   </joint>
-    <xacro:sukinee_ros2_control use_mock_hardware="$(arg use_mock_hardware)"/>
+  <xacro:sukinee_ros2_control
+    use_mock_hardware="$(arg use_mock_hardware)"
+    hardware_plugin="$(arg hardware_plugin)"
+    arm_command_interface="$(arg arm_command_interface)"
+    gripper_command_interface="$(arg gripper_command_interface)"/>
+  <xacro:if value="$(arg include_gz_plugin)">
+    <gazebo>
+      <plugin filename="gz_ros2_control-system" name="gz_ros2_control::GazeboSimROS2ControlPlugin">
+        <parameters>$(arg controllers_file)</parameters>
+      </plugin>
+    </gazebo>
+  </xacro:if>
 </robot>

Commit message: Update Sukinee robotic arm project

File: src/sukinee_urdf/urdf/sukinee_ros2_control.xacro (robot description, xacro)
@@ -1,5 +1,5 @@
 <?xml version="1.0"?>
 <robot xmlns:xacro="http://www.ros.org/wiki/xacro">
-  <xacro:macro name="sukinee_ros2_control" params="use_mock_hardware hardware_plugin arm_command_interface gripper_command_interface">
+  <xacro:macro name="sukinee_ros2_control" params="use_mock_hardware hardware_plugin arm_command_interface gripper_command_interface use_gazebo_gripper_controller">
     <ros2_control name="SukineeSystem" type="system">
     <hardware>
@@ -44,4 +44,16 @@
         <state_interface name="velocity"/>
       </joint>
+      <xacro:if value="${use_gazebo_gripper_controller}">
+        <joint name="right_finger">
+          <command_interface name="position"/>
+          <state_interface name="position"/>
+          <state_interface name="velocity"/>
+        </joint>
+        <joint name="left_finger">
+          <command_interface name="position"/>
+          <state_interface name="position"/>
+          <state_interface name="velocity"/>
+        </joint>
+      </xacro:if>
     </ros2_control>
   </xacro:macro>

File: src/sukinee_urdf/urdf/sukinee_urdf.urdf (robot description, URDF)
Before this commit: robot sukinee_urdf, 12 links, 11 joints
Links:
- removed link Link10
- removed link Link9
- added link Link_l, mass 0.034938; collision mesh filename=package://sukinee_urdf/meshes/urdf_camera_gripper/Link_l.STL; visual mesh filename=package://sukinee_urdf/meshes/urdf_camera_gripper/Link_l.STL
- added link Link_r, mass 0.034938; collision mesh filename=package://sukinee_urdf/meshes/urdf_camera_gripper/Link_r.STL; visual mesh filename=package://sukinee_urdf/meshes/urdf_camera_gripper/Link_r.STL
- added link tool0
- link Link1: mass 0.173656729959474 -> 0.37961; geometry collision mesh filename=package://sukinee_urdf/meshes/urdf_camera_gripper/Link1.STL; visual mesh filename=package://sukinee_urdf/meshes/urdf_camera_gripper/Link1.STL
- link Link2: mass 0.486273817491279 -> 0.63265; geometry collision mesh filename=package://sukinee_urdf/meshes/urdf_camera_gripper/Link2.STL; visual mesh filename=package://sukinee_urdf/meshes/urdf_camera_gripper/Link2.STL
- link Link3: mass 0.324306511251341 -> 0.50027; geometry collision mesh filename=package://sukinee_urdf/meshes/urdf_camera_gripper/Link3.STL; visual mesh filename=package://sukinee_urdf/meshes/urdf_camera_gripper/Link3.STL
- link Link4: mass 0.058588375547201 -> 0.27416; geometry collision mesh filename=package://sukinee_urdf/meshes/urdf_camera_gripper/Link4.STL; visual mesh filename=package://sukinee_urdf/meshes/urdf_camera_gripper/Link4.STL
- link Link5: mass 0.0484344180023895 -> 0.23438; geometry collision mesh filename=package://sukinee_urdf/meshes/urdf_camera_gripper/Link5.STL; visual mesh filename=package://sukinee_urdf/meshes/urdf_camera_gripper/Link5.STL
- link Link6: mass 0.159442082245761 -> 0.25842; geometry collision mesh filename=package://sukinee_urdf/meshes/urdf_camera_gripper/Link6.STL; visual mesh filename=package://sukinee_urdf/meshes/urdf_camera_gripper/Link6.STL
- link Link7: mass 0.00564266139065291 -> 0.0027847; geometry collision mesh filename=package://sukinee_urdf/meshes/urdf_camera_gripper/Link7.STL; visual mesh filename=package://sukinee_urdf/meshes/urdf_camera_gripper/Link7.STL
- link Link8: mass 0.0196144070602556 -> 0.019614; geometry collision mesh filename=package://sukinee_urdf/meshes/urdf_camera_gripper/Link8.STL; visual mesh filename=package://sukinee_urdf/meshes/urdf_camera_gripper/Link8.STL
- link base_link: mass 0.258345451540463 -> 0.54275; geometry collision mesh filename=package://sukinee_urdf/meshes/urdf_camera_gripper/base_link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; visual mesh filename=package://sukinee_urdf/meshes/urdf_camera_gripper/base_link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
Joints:
- added joint tool0_fixed_joint: type fixed, parent Link8, child tool0, origin xyz=-0.000737 -0.000386 0.040000 rpy=0 0 0
- joint Joint1: limit effort=5 velocity=3.14 -> effort=5 velocity=5
- joint Joint2: limit lower=-0.79 upper=0.79 effort=5 velocity=3.14 -> lower=-0.3 upper=2.6 effort=5 velocity=5
- joint Joint3: limit lower=-0.79 upper=0.79 effort=5 velocity=3.14 -> lower=-2.36 upper=0.3 effort=5 velocity=5; origin xyz=0.26636 0.0076666 0 rpy=0 0 0 -> xyz=0.26466 -0.031009 0 rpy=0 0 0
- joint Joint4: limit lower=-0.79 upper=0.79 effort=1.6 velocity=3.14 -> lower=-0.8 upper=0.8 effort=1.6 velocity=5; origin xyz=-0.25125 -0.065507 -0.0039 rpy=0 0 0 -> xyz=-0.25553 -0.046044 -0.0039 rpy=0 0 0
- joint Joint5: limit lower=-0.79 upper=0.79 effort=1.6 velocity=3.14 -> lower=-0.8 upper=0.8 effort=1.6 velocity=5; origin xyz=-0.059809 -0.047874 -0.0245 rpy=1.5708 -1.448 -3.0944 -> xyz=-0.063304 -0.043146 -0.0245 rpy=1.5708 1.3765 3.112
- joint Joint6: limit effort=1.6 velocity=3.14 -> lower=-2.1 upper=2.1 effort=1.6 velocity=5; origin xyz=0.00093628 -0.019978 0.045 rpy=1.5708 0.0022273 0.046831 -> xyz=0.003658 0.019663 0.045 rpy=1.5708 0.0055167 2.9577; type continuous -> revolute
- joint Joint7: limit lower=-0.79 upper=0.79 effort=1.6 velocity=3.14 -> lower=0 upper=1.57 effort=1.6 velocity=5; origin xyz=0.0015425 0.00080701 -0.016911 rpy=0.047489 -0.090961 0 -> xyz=1.7459E-05 0.00014898 0.058 rpy=0 0 0; parent Link8 -> Link6
- joint Joint8: origin xyz=1.7949E-05 0.00014892 0.075 rpy=-0.047686 0.090858 -0.00433 -> xyz=1.7459E-05 0.00014898 0.075 rpy=0 0 0
- joint left_finger: child Link10 -> Link_l; limit lower=0 upper=0.04 effort=1 velocity=0.03 -> lower=0 upper=0.04 effort=1 velocity=0.02; mimic joint=Joint7 multiplier=0.05 offset=0 -> joint=Joint7 multiplier=0.025 offset=0; origin xyz=-0.038848 -0.01714 0.0038046 rpy=-0.41189 1.4591 0 -> xyz=-0.037949 -0.016609 0.083123 rpy=1.5708 1.5384 1.9865; parent Link8 -> Link6
- joint right_finger: child Link9 -> Link_r; limit lower=0 upper=0.04 effort=1 velocity=0.03 -> lower=0 upper=0.04 effort=1 velocity=0.02; mimic joint=Joint7 multiplier=0.05 offset=0 -> joint=Joint7 multiplier=0.025 offset=0; origin xyz=0.037374 0.016369 0.012356 rpy=-2.7297 -1.4591 3.1416 -> xyz=0.037984 0.016907 0.083123 rpy=1.5708 -1.5384 -1.1551; parent Link8 -> Link6

File: src/sukinee_urdf/urdf/sukinee_urdf.urdf.xacro (robot description, xacro)
@@ -8,629 +8,330 @@
   <xacro:arg name="controllers_file" default=""/>
   <xacro:arg name="world_z" default="0.0"/>
+  <xacro:arg name="use_gazebo_gripper_controller" default="false"/>
   <xacro:include filename="$(find sukinee_urdf)/urdf/sukinee_ros2_control.xacro"/>
-  <link name="world"/>
+  <link name="world" />
   <joint name="world_to_base_link" type="fixed">
-    <parent link="world"/>
-    <child link="base_link"/>
-    <origin xyz="0 0 $(arg world_z)" rpy="0 0 0"/>
-  </joint>
-  <link
-    name="base_link">
-    <inertial>
-      <origin
-        xyz="1.32130893254478E-07 1.0878882315303E-07 0.0145123930882944"
-        rpy="0 0 0" />
-      <mass
-        value="0.258345451540463" />
-      <inertia
-        ixx="0.000255695833262824"
-        ixy="-8.50566806153412E-06"
-        ixz="6.25989218367775E-10"
-        iyy="0.000143791450764687"
-        iyz="5.1542362971656E-10"
-        izz="0.0003184122634403" />
-    </inertial>
-    <visual>
-      <origin
-        xyz="0 0 0"
-        rpy="0 0 0" />
-      <geometry>
-        <mesh
-          filename="package://sukinee_urdf/meshes/urdf2/base_link.STL" />
-      </geometry>
-      <material
-        name="">
-        <color
-          rgba="1 1 1 1" />
-      </material>
-    </visual>
-    <collision>
-      <origin
-        xyz="0 0 0"
-        rpy="0 0 0" />
-      <geometry>
-        <mesh
-          filename="package://sukinee_urdf/meshes/urdf2/base_link.STL" />
-      </geometry>
-    </collision>
-  </link>
-  <link
-    name="Link1">
-    <inertial>
-      <origin
-        xyz="-0.00339213548156639 0.000304711073311301 0.034122625208467"
-        rpy="0 0 0" />
-      <mass
-        value="0.173656729959474" />
-      <inertia
-        ixx="8.56959788246817E-05"
-        ixy="2.57981779041257E-06"
-        ixz="7.14608803543954E-07"
-        iyy="7.07301657377921E-05"
-        iyz="1.19276284474143E-07"
-        izz="9.04237787575582E-05" />
-    </inertial>
-    <visual>
-      <origin
-        xyz="0 0 0"
-        rpy="0 0 0" />
-      <geometry>
-        <mesh
-          filename="package://sukinee_urdf/meshes/urdf2/Link1.STL" />
-      </geometry>
-      <material
-        name="">
-        <color
-          rgba="1 1 1 1" />
-      </material>
-    </visual>
-    <collision>
-      <origin
-        xyz="0 0 0"
-        rpy="0 0 0" />
-      <geometry>
-        <mesh
-          filename="package://sukinee_urdf/meshes/urdf2/Link1.STL" />
-      </geometry>
-    </collision>
-  </link>
-  <joint
-    name="Joint1"
-    type="continuous">
-    <origin
-      xyz="0 0 0.0514"
-      rpy="0 0 0" />
-    <parent
-      link="base_link" />
-    <child
-      link="Link1" />
-    <axis
-      xyz="0 0 -1" />
-    <limit
-      effort="5"
-      velocity="3.14" />
-  </joint>
-  <link
-    name="Link2">
-    <inertial>
-      <origin
-        xyz="0.164355934511196 0.0107983189121957 -0.0273278206693135"
-        rpy="0 0 0" />
-      <mass
-        value="0.486273817491279" />
-      <inertia
-        ixx="0.000131700208765616"
-        ixy="-3.59955416546668E-05"
-        ixz="-4.49796251556987E-06"
-        iyy="0.00142428639296128"
-        iyz="-7.11032579861893E-07"
-        izz="0.00143980686835948" />
-    </inertial>
-    <visual>
-      <origin
-        xyz="0 0 0"
-        rpy="0 0 0" />
-      <geometry>
-        <mesh
-          filename="package://sukinee_urdf/meshes/urdf2/Link2.STL" />
-      </geometry>
-      <material
-        name="">
-        <color
-          rgba="1 1 1 1" />
-      </material>
-    </visual>
-    <collision>
-      <origin
-        xyz="0 0 0"
-        rpy="0 0 0" />
-      <geometry>
-        <mesh
-          filename="package://sukinee_urdf/meshes/urdf2/Link2.STL" />
-      </geometry>
-    </collision>
-  </link>
-  <joint
-    name="Joint2"
-    type="revolute">
-    <origin
-      xyz="-0.010939 0.025949 0.0425"
-      rpy="-1.5708 -0.00097565 0.16603" />
-    <parent
-      link="Link1" />
-    <child
-      link="Link2" />
-    <axis
-      xyz="0 0 -1" />
-    <limit
-      lower="-0.79"
-      upper="0.79"
-      effort="5"
-      velocity="3.14" />
-  </joint>
-  <link
-    name="Link3">
-    <inertial>
-      <origin
-        xyz="-0.129522607900688 -0.0521849921825459 -0.0273613995018329"
-        rpy="0 0 0" />
-      <mass
-        value="0.324306511251341" />
-      <inertia
-        ixx="8.179700405764E-05"
-        ixy="-4.69997732333903E-05"
-        ixz="1.35034163751212E-06"
-        iyy="0.000731273265167081"
-        iyz="-3.54063317410718E-07"
-        izz="0.00075003040907452" />
-    </inertial>
-    <visual>
-      <origin
-        xyz="0 0 0"
-        rpy="0 0 0" />
-      <geometry>
-        <mesh
-          filename="package://sukinee_urdf/meshes/urdf2/Link3.STL" />
-      </geometry>
-      <material
-        name="">
-        <color
-          rgba="1 1 1 1" />
-      </material>
-    </visual>
-    <collision>
-      <origin
-        xyz="0 0 0"
-        rpy="0 0 0" />
-      <geometry>
-        <mesh
-          filename="package://sukinee_urdf/meshes/urdf2/Link3.STL" />
-      </geometry>
-    </collision>
-  </link>
-  <joint
-    name="Joint3"
-    type="revolute">
-    <origin
-      xyz="0.26636 0.0076666 0"
-      rpy="0 0 0" />
-    <parent
-      link="Link2" />
-    <child
-      link="Link3" />
-    <axis
-      xyz="0 0 -1" />
-    <limit
-      lower="-0.79"
-      upper="0.79"
-      effort="5"
-      velocity="3.14" />
-  </joint>
-  <link
-    name="Link4">
-    <inertial>
-      <origin
-        xyz="-0.0338567228905684 -0.0377615700439491 -0.0271938522907798"
-        rpy="0 0 0" />
-      <mass
-        value="0.058588375547201" />
-      <inertia
-        ixx="3.47939295698438E-05"
-        ixy="-9.83781789279702E-06"
-        ixz="8.18793872056976E-08"
-        iyy="4.43014363876168E-05"
-        iyz="1.11539635337878E-07"
-        izz="3.36963199084079E-05" />
-    </inertial>
-    <visual>
-      <origin
-        xyz="0 0 0"
-        rpy="0 0 0" />
-      <geometry>
-        <mesh
-          filename="package://sukinee_urdf/meshes/urdf2/Link4.STL" />
-      </geometry>
-      <material
-        name="">
-        <color
-          rgba="1 1 1 1" />
-      </material>
-    </visual>
-    <collision>
-      <origin
-        xyz="0 0 0"
-        rpy="0 0 0" />
-      <geometry>
-        <mesh
-          filename="package://sukinee_urdf/meshes/urdf2/Link4.STL" />
-      </geometry>
-    </collision>
-  </link>
-  <joint
-    name="Joint4"
-    type="revolute">
-    <origin
-      xyz="-0.25125 -0.065507 -0.0039"
-      rpy="0 0 0" />
-    <parent
-      link="Link3" />
-    <child
-      link="Link4" />
-    <axis
-      xyz="0 0 -1" />
-    <limit
-      lower="-0.79"
-      upper="0.79"
-      effort="1.6"
-      velocity="3.14" />
-  </joint>
-  <link
-    name="Link5">
-    <inertial>
-      <origin
-        xyz="-0.000134027999521009 0.00371921314809703 0.0379219237691387"
-        rpy="0 0 0" />
-      <mass
-        value="0.0484344180023895" />
-      <inertia
-        ixx="1.25630144061511E-05"
-        ixy="-5.6639378393227E-08"
-        ixz="2.42191466268887E-08"
-        iyy="1.45689847121451E-05"
-        iyz="-4.17273377359512E-07"
-        izz="1.52122625669006E-05" />
-    </inertial>
-    <visual>
-      <origin
-        xyz="0 0 0"
-        rpy="0 0 0" />
-      <geometry>
-        <mesh
-          filename="package://sukinee_urdf/meshes/urdf2/Link5.STL" />
-      </geometry>
-      <material
-        name="">
-        <color
-          rgba="1 1 1 1" />
-      </material>
-    </visual>
-    <collision>
-      <origin
-        xyz="0 0 0"
-        rpy="0 0 0" />
-      <geometry>
-        <mesh
-          filename="package://sukinee_urdf/meshes/urdf2/Link5.STL" />
-      </geometry>
-    </collision>
-  </link>
-  <joint
-    name="Joint5"
-    type="revolute">
-    <origin
-      xyz="-0.059809 -0.047874 -0.0245"
-      rpy="1.5708 -1.448 -3.0944" />
-    <parent
-      link="Link4" />
-    <child
-      link="Link5" />
-    <axis
-      xyz="0 0 -1" />
-    <limit
-      lower="-0.79"
-      upper="0.79"
-      effort="1.6"
-      velocity="3.14" />
-  </joint>
-  <link
-    name="Link6">
-    <inertial>
-      <origin
-        xyz="0.00409063342879451 -0.00996067616063645 0.0520352103433763"
-        rpy="0 0 0" />
-      <mass
-        value="0.159442082245761" />
-      <inertia
-        ixx="3.47012582789967E-05"
-        ixy="-4.54172618430741E-05"
-        ixz="5.33673918445066E-08"
-        iyy="0.000118901432832412"
-        iyz="-7.69611955935196E-07"
-        izz="0.000144711425342682" />
-    </inertial>
-    <visual>
-      <origin
-        xyz="0 0 0"
-        rpy="0 0 0" />
-      <geometry>
-        <mesh
-          filename="package://sukinee_urdf/meshes/urdf2/Link6.STL" />
-      </geometry>
-      <material
-        name="">
-        <color
-          rgba="1 1 1 1" />
-      </material>
-    </visual>
-    <collision>
-      <origin
-        xyz="0 0 0"
-        rpy="0 0 0" />
-      <geometry>
-        <mesh
-          filename="package://sukinee_urdf/meshes/urdf2/Link6.STL" />
-      </geometry>
-    </collision>
-  </link>
-  <joint
-    name="Joint6"
-    type="continuous">
-    <origin
-      xyz="0.00093628 -0.019978 0.045"
-      rpy="1.5708 0.0022273 0.046831" />
-    <parent
-      link="Link5" />
-    <child
-      link="Link6" />
-    <axis
-      xyz="0 0 -1" />
-    <limit
-      effort="1.6"
-      velocity="3.14" />
-  </joint>
-  <link
-    name="Link8">
-    <inertial>
-      <origin
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